File: open-semg-16-electronics/open-semg-16.kicad_sch (KiCad schematic)
At the start: 121 parts, among them J1 Reference Electrode, J2 Reference Electrode, U1 ADS1298xPAG, U2 ADS1298xPAG, U4 LP2985-3.3, U6 ESP32-S3-WROOM-1, U7 TLV75533PDBV

Commit message: Update RLD Configuration for both ADCs
Parts:
- renumbered J2 to J1, U2 to U1, U1 to U2
Connections:
- net at C1.1, J1.1 (Pin_1), R1.1: no longer U2.63 (RLDOUT)
Other:
- moved on the sheet: BT1, C1, C11, C13, C14, C15, C17, C18, C19, C2, C20, C21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
