File: open-semg-8-electronics/_autosave-open-semg-8.kicad_sch (KiCad schematic)
At the start: 67 parts, among them J1 Reference Electrode, U1 ADS1298xPAG, U4 LP2985-3.3, U6 ESP32-S3-WROOM-1, U7 TLV75533PDBV

Commit message: Update smeg-8 channels schematics
Connections:
- net DAISY_CHAIN_B is gone; now on net MISO: U1.43 (DOUT)
- net DRDY: now also U1.47 (~{DRDY})
Other:
- moved on the sheet: BT1, C1, C11, C17, C18, C19, C2, C20, C21, C26, C27, C28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
