File: open-semg-8-electronics/open-semg-8.kicad_sch (KiCad schematic)
At the start: 121 parts, among them J1 Reference Electrode, J2 Reference Electrode, U1 ADS1298xPAG, U2 ADS1298xPAG, U4 LP2985-3.3, U6 ESP32-S3-WROOM-1, U7 TLV75533PDBV

Commit message: Update 8-channel schematic
Parts:
- removed C13, C14, C15, C50, C51, C52, C53, C54, C55, C56, C57, C58, C59, C60, C61, C62: 620pF, symbol Device:C
- removed C63: 22uF, symbol Device:C
- removed C64, C65, C66: 1uF, symbol Device:C
- removed C67, C69, C71: 0.1uF, symbol Device:C
- removed C68, C70, C72: 10uF, symbol Device:C
- removed C73: 1.5nF, symbol Device:C
- removed E17, E18, E19, E20, E21, E22, E23, E24: Electrodes, symbol Connector:Conn_01x02_Pin
- removed J2: Reference Electrode, symbol Connector:Conn_01x01_Pin
- removed R21, R22, R23, R24, R25, R26, R27, R28, R29, R3, R30, R31, R32, R33, R34, R35: 2KΩ, symbol Device:R
- removed R36: 1MΩ, symbol Device:R
- removed U2: ADS1298xPAG, Package_QFP:TQFP-64_10x10mm_P0.5mm, symbol Analog_ADC:ADS1298xPAG
Connections:
- net DAISY_CHAIN_B is gone; now on net MISO: U1.43 (DOUT)
- net DRDY: now also U1.47 (~{DRDY})
- no-connect marks 6 -> 3
Other:
- moved on the sheet: BT1, C1, C11, C17, C18, C19, C2, C20, C21, C26, C27, C28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
