File: open-semg-16-v1/open-semg-16-v1.kicad_sch (KiCad schematic)
At the start: 111 parts, among them U1 ADS1298xPAG, U2 ADS1298xPAG, U3 ESP32-S3-DevKitC, U4 LP2985-3.3, U5 TLV75533PDBV

Commit message: some fixes for ambrflow suggestions
Connections:
- no-connect marks 9 -> 37
Changed lines of the file:
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@@
 	)
 	(no_connect
+		(at 562.61 101.6)
+	)
+	(no_connect
+		(at 562.61 66.04)
+	)
+	(no_connect
+		(at 562.61 124.46)
+	)
+	(no_connect
+		(at 562.61 121.92)
+	)
+	(no_connect
+		(at 562.61 109.22)
+	)
+	(no_connect
+		(at 562.61 99.06)
+	)
+	(no_connect
 		(at 195.58 106.68)
 	)
 	(no_connect
+		(at 562.61 104.14)
+	)
+	(no_connect
+		(at 562.61 63.5)
+	)
+	(no_connect
+		(at 511.81 53.34)
+	)
+	(no_connect
+		(at 511.81 66.04)
+	)
+	(no_connect
 		(at 195.58 116.84)
 	)
 	(no_connect
+		(at 511.81 63.5)
+	)
+	(no_connect
 		(at 422.91 163.83)
 	)
 	(no_connect
+		(at 511.81 68.58)
+	)
+	(no_connect
+		(at 562.61 114.3)
+	)
+	(no_connect
 		(at 422.91 107.95)
 	)
 	(no_connect
+		(at 562.61 111.76)
+	)
+	(no_connect
+		(at 562.61 119.38)
+	)
+	(no_connect
+		(at 562.61 45.72)
+	)
+	(no_connect
 		(at 422.91 113.03)
 	)
 	(no_connect
+		(at 562.61 53.34)
+	)
+	(no_connect
+		(at 562.61 116.84)
+	)
+	(no_connect
 		(at 422.91 115.57)
 	)
@@
 	)
 	(no_connect
+		(at 562.61 60.96)
+	)
+	(no_connect
 		(at 422.91 105.41)
 	)
 	(no_connect
+		(at 511.81 43.18)
+	)
+	(no_connect
+		(at 562.61 50.8)
+	)
+	(no_connect
+		(at 511.81 50.8)
+	)
+	(no_connect
+		(at 511.81 60.96)
+	)
+	(no_connect
 		(at 195.58 109.22)
 	)
+	(no_connect
+		(at 562.61 43.18)
+	)
+	(no_connect
+		(at 562.61 68.58)
+	)
+	(no_connect
+		(at 562.61 106.68)
+	)
+	(no_connect
+		(at 562.61 73.66)
+	)
+	(no_connect
+		(at 562.61 71.12)
+	)
 	(wire
 		(pts
@@
 	(wire
 		(pts
+			(xy 144.78 266.7) (xy 144.78 267.97)
+		)
+		(stroke
+			(width 0)
+			(type default)
+		)
+	)
+	(wire
+		(pts
 			(xy 364.49 189.23) (xy 364.49 186.69)
 		)
@@
 	(wire
 		(pts
+			(xy 147.32 267.97) (xy 147.32 269.24)
+		)
+		(stroke
+			(width 0)
+			(type default)
+		)
+	)
+	(wire
+		(pts
 			(xy 276.86 66.04) (xy 283.21 66.04)
 		)
@@
 	(wire
 		(pts
+			(xy 144.78 267.97) (xy 147.32 267.97)
+		)
+		(stroke
+			(width 0)
+			(type default)
+		)
+	)
+	(wire
+		(pts
 			(xy 307.34 158.75) (xy 309.88 158.75)
 		)
@@
 		)
 	)
+	(label "AVDD"
+		(at 144.78 266.7 0)
+		(effects
+			(font
+				(size 1.27 1.27)
+			)
+			(justify left bottom)
+		)
+	)
 	(label "DVDD"
 		(at 209.55 160.02 180)
@@
 		(property "Value" "+3.3V"
 			(at 147.32 264.16 0)
+			(hide yes)
 			(show_name no)
 			(do_not_autoplace no)
