File: open-semg-16-v1-codex/v1.2/open-semg-16-v1.2.kicad_sch (KiCad schematic)
At the start: 130 parts, among them U1 ADS1298xPAG, U2 ADS1298xPAG, U3 ESP32-S3-DevKitC, U4 LP2985-3.3, U5 TLV75533PDBV

Commit message: some fixes for ambrflow suggestions
Parts:
- added R36, R37: 10k, symbol Device:R
- added R38: 0, symbol Device:R
- C1, C10, C11, C12, C13, C14, C15, C16, C17, C18, C2, C21, C22, C27, C28, C29, C3, C30, C31, C36, C37, C38, C39, C4, C40, C41, C42, C43, C44, C47, C48, C5: Dielectric (none) -> C0G/NP0; Qualification (none) -> F12/F14: matched input RC; component requirements only, ele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; Tolerance (none) -> 1%
- C25, C51: Qualification (none) -> F14: qualify selected 1uF part at VCAP3 bias (~5.2V at 3.3V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; Voltage rating (none) -> >=10 V
- C55: Leakage current (none) -> <100 nA at operating bias and temperature; Qualification (none) -> F14: LP2985 section 7.1.3; retain 10nF BP bypass; exact MPN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
- R1, R10, R11, R12, R13, R14, R15, R16, R17, R18, R19, R2, R20, R21, R22, R23, R24, R25, R26, R27, R28, R29, R3, R30, R31, R32, R4, R5, R6, R7, R8, R9: Qualification (none) -> F12/F14: preserve 2k input topology; resistor rating does n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; Rated power (none) -> >=0.1 W; verify temperature derating and fault pulses; Tolerance (none) -> 0.1%
Connections:
- net +3.3V: no longer C54.1, U4.5 (VOUT)
- net AGND: now also R36.2, R37.2, R38.2
- net EN: now also R38.1
- net MOSI: now also R36.1
- net SCLK: now also R37.1
- new net LP2985_OUT_DISABLED: C54.1, U4.5 (VOUT)
- no-connect marks 8 -> 34
Other:
- note added: "F04: U4 output isolated with C54; no system load. Both LDOs remain OFF. Qualify LP silicon/C54 before enable."
- note added: "V1.2 F09: R36/R37 bias DIN and SCLK low; CS / full sequencing unresolved. F05: R38 = 0R FITTED: both LDOs held OFF. No functional enable source. Keep R38 fitted until functional EN, F13/F15/F16/F17 qualification is complete. USB / external +3.3V can still backfeed the rail; OFF strap is not isolation."
- note added: "V1.2 F12/F14 - PROCUREMENT REQUIREMENTS (not qualified installed parts) R1-R32: 2k unchanged; 0.1%, >=0.1W, derating/pulse review required. All 32 input 620pF caps: C0G/NP0, 1%; electrode impedance/CMRR still unverified. C25/C51 VCAP3: 1uF unchanged, >=10V; qualify capacitance at ~5.2V DC. C55 BP: 10nF unchanged; leakage <100nA at operating bias/temperature. No MPN, footprint, physical performanc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"
- note added: "V1.2 PARTIAL CORRECTIONS - NOT READY FOR POWER-UP OR WEARER USE F04: U4/C54 isolated from main rail. F05: R38 holds both LDOs OFF; operating power unqualified. F06/F18: restore U1 CLK_EN after RESET; allow U2 clock/POR; configure before shared START. F09: START/RESET/PWDN plus DIN/SCLK have pulldowns; CS/full sequencing unresolved. Enable/settle 2.4V reference; verify gain/rate; keep PACE/RLD/WCT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"
- note removed: "V2 PARTIAL CORRECTIONS - NOT READY FOR POWER-UP OR WEARER USE F04/F05: parallel LDO outputs and floating EN remain; power architecture requires approval. F06/F18: restore U1 CLK_EN after RESET; allow U2 clock/POR; configure both before shared START. F09: START/RESET/PWDN biased low while MCU is high-Z; CS defaults and full sequencing remain unresolved. Enable/settle 2.4V reference; verify gain/ra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"
